File: pcb/PDB.kicad_pcb (KiCad board)
At the start: 2 copper layers, 77.5 x 50.8 mm, 120 parts, among them J1 USB_C_Receptacle, J2 Conn_02x02_Counter_Clockwise, J3 Conn_02x02_Counter_Clockwise, J4 Conn_02x02_Counter_Clockwise, J5 Conn_02x02_Counter_Clockwise, J6 Conn_01x03_Pin, J7 Conn_01x03_Pin, SW1 SW_Push, SW2 SW_DIP_x02, U1 BD81870EFV-ME2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

Commit message: Update to KiCAD 9
Parts:
- D1, D2: value DO-214AC -> DO-214AC
- U10, U11: footprint Package_TO_SOT_SMD:TO-252-3_TabPin2 -> Package_TO_SOT_SMD:TO-252-2
