File: pcb/PDB.kicad_pcb (KiCad board)
At the start: 2 copper layers, 77.5 x 50.8 mm, 120 parts, among them J1 USB_C_Receptacle, J2 Conn_02x02_Counter_Clockwise, J3 Conn_02x02_Counter_Clockwise, J4 Conn_02x02_Counter_Clockwise, J5 Conn_02x02_Counter_Clockwise, J6 Conn_01x03_Pin, J7 Conn_01x03_Pin, SW1 SW_Push, SW2 SW_DIP_x02, U1 BD81870EFV-ME2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

Commit message: Change MCP2221A to FT230X
Parts:
- removed C27: 10n, Capacitor_SMD:C_1206_3216Metric
- removed R30: 1k, Resistor_SMD:R_1206_3216Metric
- U13: value MCP2221AxSL -> FT230XS; footprint Package_SO:SOIC-14_3.9x8.7mm_P1.27mm -> Package_SO:SSOP-16_3.9x4.9mm_P0.635mm
- moved FID2 14.8 mm to (125.8, 90.8)
- moved C23 6.83 mm to (139.9, 100.2), turned to 90 degrees
- moved C21 4.14 mm to (134.9, 96.7), turned to 180 degrees
- moved U13 1.95 mm to (135.5, 101.6), turned to -90 degrees
- moved R36 0.64 mm to (134.2, 109.7)
- moved R37 0.64 mm to (134.2, 107.2)
- moved D7 0.52 mm to (129.2, 109.7)
- moved D8 0.52 mm to (129.2, 107.2)
Connections:
- C21 pad 1: Net-(U13-VUSB) -> +3V3
- D7 pad 2: +5V -> +3V3
- D8 pad 2: +5V -> +3V3
- R31 pad 2: Net-(U13-URx) -> Net-(U13-RXD)
- R32 pad 2: Net-(U13-D+) -> Net-(U13-USBDP)
- R33 pad 2: Net-(U13-UTx) -> Net-(U13-TXD)
- R35 pad 2: Net-(U13-D-) -> Net-(U13-USBDM)
- R36 pad 2: Net-(U13-GP0) -> Net-(U13-CBUS0)
- R37 pad 2: Net-(U13-GP1) -> Net-(U13-CBUS1)
- SW2 pad 1: Net-(U13-UTx) -> Net-(U13-TXD)
- SW2 pad 2: Net-(U13-URx) -> Net-(U13-RXD)
- U13 pad 1: +5V -> Net-(U13-TXD)
- U13 pad 10: unconnected-(U13-SCL-Pad10) -> +3V3
- U13 pad 11: Net-(U13-VUSB) -> +3V3
- U13 pad 12: Net-(U13-D-) -> +5V
- U13 pad 13: Net-(U13-D+) -> GND
- U13 pad 14: GND -> Net-(U13-CBUS1)
- U13 pad 2: Net-(U13-GP0) -> unconnected-(U13-~{RTS}-Pad2)
- U13 pad 3: Net-(U13-GP1) -> +3V3
- U13 pad 4: Net-(U13-~{RST}) -> Net-(U13-RXD)
- U13 pad 5: Net-(U13-URx) -> GND
- U13 pad 6: Net-(U13-UTx) -> unconnected-(U13-~{CTS}-Pad6)
- U13 pad 8: unconnected-(U13-GP3-Pad8) -> Net-(U13-USBDP)
- U13 pad 9: unconnected-(U13-SDA-Pad9) -> Net-(U13-USBDM)
Routing:
- net +5V: track 130.2 -> 102.6 mm, vias 32 -> 31
- net Net-(U13-UTx): track 25.0 -> 0.00 mm, vias 2 -> 0
- net Net-(U13-TXD): track 0.00 -> 22.3 mm, vias 0 -> 2
- net Net-(U13-URx): track 22.2 -> 0.00 mm, vias 2 -> 0
- net +3V3: track 0.00 -> 20.6 mm, vias 0 -> 2
- net Net-(U13-RXD): track 0.00 -> 19.4 mm, vias 0 -> 2
- net Net-(U13-GP0): track 8.98 -> 0.00 mm
- net Net-(U13-GP1): track 8.08 -> 0.00 mm
- net Net-(U13-CBUS0): track 0.00 -> 6.13 mm
- net Net-(U13-USBDM): track 0.00 -> 5.51 mm, vias 0 -> 2
- net Net-(U13-USBDP): track 0.00 -> 5.50 mm
- net Net-(U13-~{RST}): track 5.02 -> 0.00 mm
- net Net-(U13-VUSB): track 3.93 -> 0.00 mm
- net Net-(U13-CBUS1): track 0.00 -> 3.33 mm
- net Net-(U13-D-): track 3.10 -> 0.00 mm
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
Commit message: Optimize +3V3 signal
Connections:
- net +3V3 renamed Net-(D7-A)
Changed lines of the file:
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@@
 	(net 71 "unconnected-(U12-PA5-Pad3)")
 	(net 72 "Net-(U3-OUT)")
-	(net 73 "+3V3")
+	(net 73 "Net-(D7-A)")
 	(net 74 "Net-(U13-RXD)")
 	(net 75 "Net-(U13-USBDP)")
@@
 			(layers "F.Cu" "F.Mask" "F.Paste")
 			(roundrect_rratio 0.2)
-			(net 73 "+3V3")
+			(net 73 "Net-(D7-A)")
 			(pinfunction "A")
 			(pintype "passive")
@@
 			(size 1.2 0.4)
 			(layers "F.Cu" "F.Mask" "F.Paste")
-			(net 73 "+3V3")
+			(net 73 "Net-(D7-A)")
 			(pinfunction "VCCIO")
 			(pintype "power_in")
@@
 			(size 1.2 0.4)
 			(layers "F.Cu" "F.Mask" "F.Paste")
-			(net 73 "+3V3")
+			(net 73 "Net-(D7-A)")
 			(pinfunction "3V3OUT")
 			(pintype "power_out")
@@
 			(size 1.2 0.4)
 			(layers "F.Cu" "F.Mask" "F.Paste")
-			(net 73 "+3V3")
+			(net 73 "Net-(D7-A)")
 			(pinfunction "~{RESET}")
 			(pintype "input")
@@
 			(layers "F.Cu" "F.Mask" "F.Paste")
 			(roundrect_rratio 0.2)
-			(net 73 "+3V3")
+			(net 73 "Net-(D7-A)")
 			(pinfunction "A")
 			(pintype "passive")
@@
 			(layers "F.Cu" "F.Mask" "F.Paste")
 			(roundrect_rratio 0.217391)
-			(net 73 "+3V3")
+			(net 73 "Net-(D7-A)")
 			(pintype "passive")
 		)
