File: pcb/PDB.kicad_sch (KiCad schematic)
At the start: 84 parts, among them J1 USB_C_Receptacle, J2 Conn_02x02_Counter_Clockwise, J3 Conn_02x02_Counter_Clockwise, J4 Conn_02x02_Counter_Clockwise, J5 Conn_02x02_Counter_Clockwise, J6 Conn_01x03_Pin, J7 Conn_01x03_Pin, U1 BD81870EFV-ME2, U10 LM337_TO252, U11 LM317_TO-252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

Commit message: Update to KiCAD 9
Parts:
- C1, C17, C18, C19, C2, C20, C4: DigiKey (none) -> 732-8545-1-ND; Vendor DigiKey -> (none); VendorId 732-8545-1-ND -> (none)
- C10, C11, C16, C5: HTL (none) -> 100138; Vendor HTL -> (none); VendorId 100138 -> (none)
- C12: HTL (none) -> 100105; Vendor HTL -> (none); VendorId 100105 -> (none)
- C13: HTL (none) -> 100108; Vendor HTL -> (none); VendorId 100108 -> (none)
- C14, C28, C6, C7, C8, C9: HTL (none) -> 100128; Vendor HTL -> (none); VendorId 100128 -> (none)
- C15, C3: HTL (none) -> 100134; Vendor HTL -> (none); VendorId 100134 -> (none)
- D1, D2: value DO-214AC -> DO-214AC; HTL (none) -> 103360; Vendor HTL -> (none); VendorId 103360 -> (none)
- D3: HTL (none) -> 100193; Vendor HTL -> (none); VendorId 100193 -> (none)
- D4, D5: HTL (none) -> 103360; Vendor HTL -> (none); VendorId 103360 -> (none)
- F1: HTL (none) -> 103597; Vendor HTL -> (none); VendorId 103597 -> (none)
- FB1: HTL (none) -> 103570; Vendor HTL -> (none); VendorId 103570 -> (none)
- FID1, FID2, FID3, FID4: now left out of the parts list
- H1, H2, H3, H4: HTL (none) -> 101179; Vendor HTL -> (none); VendorId 101179 -> (none)
- J1: HTL (none) -> 103572; Vendor HTL -> (none); VendorId 103572 -> (none)
- J2, J3, J4, J5: DigiKey (none) -> 2057-RS2-04-G-ND; Vendor DigiKey -> (none); VendorId 2057-RS2-04-G-ND -> (none)
- J6, J7: HTL (none) -> 101521; Vendor HTL -> (none); VendorId 101521 -> (none)
- L1, L2: DigiKey (none) -> 587-2893-1-ND; Vendor DigiKey -> (none); VendorId 587-2893-1-ND -> (none)
- R1, R2, R4: HTL (none) -> 102962; Vendor HTL -> (none); VendorId 102962 -> (none)
- R10: HTL (none) -> 102970; Vendor HTL -> (none); VendorId 102970 -> (none)
- R11: HTL (none) -> 102951; Vendor HTL -> (none); VendorId 102951 -> (none)
- R12: HTL (none) -> 102952; Vendor HTL -> (none); VendorId 102952 -> (none)
- R13, R14: HTL (none) -> 102955; Vendor HTL -> (none); VendorId 102955 -> (none)
- R15, R17, R25, R26, R9: HTL (none) -> 102966; Vendor HTL -> (none); VendorId 102966 -> (none)
- R20, R21: DigiKey (none) -> CRM2010-FX-R100ELFCT-ND; Vendor DigiKey -> (none); VendorId CRM2010-FX-R100ELFCT-ND -> (none)
- R22: HTL (none) -> 103577; Vendor HTL -> (none); VendorId 103577 -> (none)
- R23: HTL (none) -> 102958; Vendor HTL -> (none); VendorId 102958 -> (none)
- R24: HTL (none) -> 102949; Vendor HTL -> (none); VendorId 102949 -> (none)
- R3: HTL (none) -> 102989; Vendor HTL -> (none); VendorId 102989 -> (none)
- R5: HTL (none) -> 102988; Vendor HTL -> (none); VendorId 102988 -> (none)
- R6: HTL (none) -> 102967; Vendor HTL -> (none); VendorId 102967 -> (none)
- R7: HTL (none) -> 103010; Vendor HTL -> (none); VendorId 103010 -> (none)
- R8: HTL (none) -> 102902; Vendor HTL -> (none); VendorId 102902 -> (none)
- RV1, RV2: HTL (none) -> 100424; Vendor HTL -> (none); VendorId 100424 -> (none)
- U1: DigiKey (none) -> BD81870EFV-ME2CT-ND; Vendor DigiKey -> (none); VendorId BD81870EFV-ME2CT-ND -> (none)
- U10: footprint Package_TO_SOT_SMD:TO-252-3_TabPin2 -> Package_TO_SOT_SMD:TO-252-2; DigiKey (none) -> 296-21578-1-ND; Vendor DigiKey -> (none); VendorId 296-21578-1-ND -> (none)
- U11: footprint Package_TO_SOT_SMD:TO-252-3_TabPin2 -> Package_TO_SOT_SMD:TO-252-2; DigiKey (none) -> 5272-LM317MDT-EVCT-ND; Vendor DigiKey -> (none); VendorId 5272-LM317MDT-EVCT-ND -> (none)
- U2: DigiKey (none) -> LM321SN3T1GOSCT-ND; Vendor DigiKey -> (none); VendorId LM321SN3T1GOSCT-ND -> (none)
- U3: HTL (none) -> 103270; Vendor HTL -> (none); VendorId 103270 -> (none)
- U4, U6, U8: DigiKey (none) -> 5399-TL431CT-ND; Vendor DigiKey -> (none); VendorId 5399-TL431CT-ND -> (none)
- U5, U7, U9: HTL (none) -> 103581; Vendor HTL -> (none); VendorId 103581 -> (none)
