File: pcb/PDB.kicad_sch (KiCad schematic)
At the start: 84 parts, among them J1 USB_C_Receptacle, J2 Conn_02x02_Counter_Clockwise, J3 Conn_02x02_Counter_Clockwise, J4 Conn_02x02_Counter_Clockwise, J5 Conn_02x02_Counter_Clockwise, J6 Conn_01x03_Pin, J7 Conn_01x03_Pin, U1 BD81870EFV-ME2, U10 LM337_TO252, U11 LM317_TO-252, U2 LM321, U3 L78L05_SOT89, U4 TL431DBZ, U5 INA181, U6 TL431DBZ, U7 INA181, U8 TL431DBZ, U9 INA181

Commit message: Fix wrong part-id
Parts:
- U3: HTL 103270 -> 103557
Changed lines of the file:
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@@
 			)
 		)
-		(property "HTL" "103270"
+		(property "HTL" "103557"
 			(at 116.84 92.71 0)
 			(effects

Commit message: Modify voltage divider and silkscreen
Parts:
- R23: value 2k7 -> 1k8; HTL 102958 -> 102955
- R24: value 750 -> 634; HTL 102949 -> 102947
- R25: value 8k2 -> 5k1; HTL 102966 -> 102962
- R26: value 8k2 -> 6k8; HTL 102966 -> 102964
Changed lines of the file:
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@@
 			)
 		)
-		(property "Value" "2k7"
+		(property "Value" "1k8"
 			(at 128.27 129.54 0)
 			(effects
@@
 			)
 		)
-		(property "HTL" "102958"
+		(property "HTL" "102955"
 			(at 127 130.81 0)
 			(effects
@@
 			)
 		)
-		(property "Value" "8k2"
+		(property "Value" "6k8"
 			(at 180.34 142.24 0)
 			(effects
@@
 			)
 		)
-		(property "HTL" "102966"
+		(property "HTL" "102964"
 			(at 181.61 143.51 0)
 			(effects
@@
 			)
 		)
-		(property "Value" "8k2"
+		(property "Value" "5k1"
 			(at 113.03 142.24 0)
 			(effects
@@
 			)
 		)
-		(property "HTL" "102966"
+		(property "HTL" "102962"
 			(at 114.3 143.51 0)
 			(effects
@@
 			)
 		)
-		(property "Value" "750"
+		(property "Value" "634"
 			(at 195.58 132.08 0)
 			(effects
@@
 			)
 		)
-		(property "HTL" "102949"
+		(property "HTL" "102947"
 			(at 194.31 130.81 0)
 			(effects
