File: pcb/PDB_control.kicad_sch (KiCad schematic)
At the start: 34 parts, among them SW1 SW_Push, SW2 SW_DIP_x02, U12 ATtiny1606-S, U13 FT230XS

Commit message: Update +15V voltage divider resistor values
Parts:
- R40: value 18k -> 6k8; HTL 102971 -> 102964
- R43: value 6k8 -> 2k2; HTL 102964 -> 102956
Changed lines of the file:
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@@
 			)
 		)
-		(property "Value" "6k8"
+		(property "Value" "2k2"
 			(at 82.55 161.29 90)
 			(effects
@@
 			)
 		)
-		(property "HTL" "102964"
+		(property "HTL" "102956"
 			(at 80.01 161.29 90)
 			(effects
@@
 			)
 		)
-		(property "Value" "18k"
+		(property "Value" "6k8"
 			(at 82.55 151.13 90)
 			(effects
@@
 			)
 		)
-		(property "HTL" "102971"
+		(property "HTL" "102964"
 			(at 80.01 151.13 90)
 			(effects
